Commit message: Renamed the joints

File: src/ogmen_description/urdf/ogmen.xacro (robot description, xacro)
@@ -103,5 +103,5 @@
   </collision>
 </link>
-<joint name="Revolute 1" type="continuous">
+<joint name="right_wheel_joint" type="continuous">
   <origin xyz="-0.035 -0.105 0.065" rpy="0 0 0"/>
   <parent link="base_link"/>
@@ -109,5 +109,5 @@
   <axis xyz="0.0 -1.0 0.0"/>
 </joint>
-<joint name="Revolute 2" type="continuous">
+<joint name="left_wheel_joint" type="continuous">
   <origin xyz="-0.035 0.105 0.065" rpy="0 0 0"/>
   <parent link="base_link"/>
@@ -115,10 +115,10 @@
   <axis xyz="0.0 1.0 0.0"/>
 </joint>
-<joint name="Rigid 3" type="fixed">
+<joint name="lidar_joint" type="fixed">
   <origin xyz="0.0 0.0 0.135" rpy="0 0 0"/>
   <parent link="base_link"/>
   <child link="lidar_1"/>
 </joint>
-<joint name="Rigid 4" type="fixed">
+<joint name="camera_joint" type="fixed">
   <origin xyz="0.1 0.0 0.08" rpy="0 0 0"/>
   <parent link="base_link"/>
