Commit message: update

File: src/ogmen_description/urdf/materials.xacro (robot description, xacro)
@@ -1,12 +1,6 @@
 <?xml version="1.0" ?>
 <robot name="ogmen" xmlns:xacro="http://www.ros.org/wiki/xacro" >
-<material name="silver_default">
+<material name="silver">
   <color rgba="0.700 0.700 0.700 1.000"/>
 </material>
-<material name="pa_12_nylon_pa_603cf_with_eos_p_3d_printers">
-  <color rgba="0.24705882352941178 0.24705882352941178 0.24705882352941178 1.0"/>
-</material>
-<material name="polymide_kapton">
-  <color rgba="0.7843137254901961 0.5568627450980392 0.027450980392156862 1.0"/>
-</material>
 </robot>

File: src/ogmen_description/urdf/ogmen.xacro (robot description, xacro)
@@ -3,4 +3,5 @@
 <xacro:include filename="$(find ogmen_description)/urdf/materials.xacro" />
 <xacro:include filename="$(find ogmen_description)/urdf/ogmen.trans" />
+<xacro:include filename="$(find ogmen_description)/urdf/ogmen.gazebo" />
 <link name="base_link">
   <inertial>
@@ -12,12 +13,12 @@
     <origin xyz="0 0 0" rpy="0 0 0"/>
     <geometry>
-      <mesh filename="package://ogmen_description/meshes/base_link.stl" scale="0.001 0.001 0.001"/>
+      <mesh filename="file://$(find ogmen_description)/meshes/base_link.stl" scale="0.001 0.001 0.001"/>
     </geometry>
-    <material name="pa_12_nylon_pa_603cf_with_eos_p_3d_printers"/>
+    <material name="silver"/>
   </visual>
   <collision>
     <origin xyz="0 0 0" rpy="0 0 0"/>
     <geometry>
-      <mesh filename="package://ogmen_description/meshes/base_link.stl" scale="0.001 0.001 0.001"/>
+      <mesh filename="file://$(find ogmen_description)/meshes/base_link.stl" scale="0.001 0.001 0.001"/>
     </geometry>
   </collision>
@@ -32,12 +33,12 @@
     <origin xyz="0.035 0.105 -0.065" rpy="0 0 0"/>
     <geometry>
-      <mesh filename="package://ogmen_description/meshes/right_wheel_1.stl" scale="0.001 0.001 0.001"/>
+      <mesh filename="file://$(find ogmen_description)/meshes/right_wheel_1.stl" scale="0.001 0.001 0.001"/>
     </geometry>
-    <material name="pa_12_nylon_pa_603cf_with_eos_p_3d_printers"/>
+    <material name="silver"/>
   </visual>
   <collision>
     <origin xyz="0.035 0.105 -0.065" rpy="0 0 0"/>
     <geometry>
-      <mesh filename="package://ogmen_description/meshes/right_wheel_1.stl" scale="0.001 0.001 0.001"/>
+      <mesh filename="file://$(find ogmen_description)/meshes/right_wheel_1.stl" scale="0.001 0.001 0.001"/>
     </geometry>
   </collision>
@@ -52,12 +53,12 @@
     <origin xyz="0.035 -0.105 -0.065" rpy="0 0 0"/>
     <geometry>
-      <mesh filename="package://ogmen_description/meshes/left_wheel_1.stl" scale="0.001 0.001 0.001"/>
+      <mesh filename="file://$(find ogmen_description)/meshes/left_wheel_1.stl" scale="0.001 0.001 0.001"/>
     </geometry>
-    <material name="pa_12_nylon_pa_603cf_with_eos_p_3d_printers"/>
+    <material name="silver"/>
   </visual>
   <collision>
     <origin xyz="0.035 -0.105 -0.065" rpy="0 0 0"/>
     <geometry>
-      <mesh filename="package://ogmen_description/meshes/left_wheel_1.stl" scale="0.001 0.001 0.001"/>
+      <mesh filename="file://$(find ogmen_description)/meshes/left_wheel_1.stl" scale="0.001 0.001 0.001"/>
     </geometry>
   </collision>
@@ -72,12 +73,12 @@
     <origin xyz="-0.0 -0.0 -0.135" rpy="0 0 0"/>
     <geometry>
-      <mesh filename="package://ogmen_description/meshes/lidar_1.stl" scale="0.001 0.001 0.001"/>
+      <mesh filename="file://$(find ogmen_description)/meshes/lidar_1.stl" scale="0.001 0.001 0.001"/>
     </geometry>
-    <material name="polymide_kapton"/>
+    <material name="silver"/>
   </visual>
   <collision>
     <origin xyz="-0.0 -0.0 -0.135" rpy="0 0 0"/>
     <geometry>
-      <mesh filename="package://ogmen_description/meshes/lidar_1.stl" scale="0.001 0.001 0.001"/>
+      <mesh filename="file://$(find ogmen_description)/meshes/lidar_1.stl" scale="0.001 0.001 0.001"/>
     </geometry>
   </collision>
@@ -92,16 +93,16 @@
     <origin xyz="-0.1 -0.0 -0.08" rpy="0 0 0"/>
     <geometry>
-      <mesh filename="package://ogmen_description/meshes/camera_1.stl" scale="0.001 0.001 0.001"/>
+      <mesh filename="file://$(find ogmen_description)/meshes/camera_1.stl" scale="0.001 0.001 0.001"/>
     </geometry>
-    <material name="pa_12_nylon_pa_603cf_with_eos_p_3d_printers"/>
+    <material name="silver"/>
   </visual>
   <collision>
     <origin xyz="-0.1 -0.0 -0.08" rpy="0 0 0"/>
     <geometry>
-      <mesh filename="package://ogmen_description/meshes/camera_1.stl" scale="0.001 0.001 0.001"/>
+      <mesh filename="file://$(find ogmen_description)/meshes/camera_1.stl" scale="0.001 0.001 0.001"/>
     </geometry>
   </collision>
 </link>
-<joint name="right_wheel_joint" type="continuous">
+<joint name="Revolute 1" type="continuous">
   <origin xyz="-0.035 -0.105 0.065" rpy="0 0 0"/>
   <parent link="base_link"/>
@@ -109,5 +110,5 @@
   <axis xyz="0.0 -1.0 0.0"/>
 </joint>
-<joint name="left_wheel_joint" type="continuous">
+<joint name="Revolute 2" type="continuous">
   <origin xyz="-0.035 0.105 0.065" rpy="0 0 0"/>
   <parent link="base_link"/>
@@ -115,10 +116,10 @@
   <axis xyz="0.0 1.0 0.0"/>
 </joint>
-<joint name="lidar_joint" type="fixed">
+<joint name="Rigid 3" type="fixed">
   <origin xyz="0.0 0.0 0.135" rpy="0 0 0"/>
   <parent link="base_link"/>
   <child link="lidar_1"/>
 </joint>
-<joint name="camera_joint" type="fixed">
+<joint name="Rigid 4" type="fixed">
   <origin xyz="0.1 0.0 0.08" rpy="0 0 0"/>
   <parent link="base_link"/>

Commit message: added all scripts

File: src/ogmen_description/urdf/materials.xacro (robot description, xacro)
@@ -4,3 +4,27 @@
   <color rgba="0.700 0.700 0.700 1.000"/>
 </material>
+<material name="black">
+  <color rgba="0.0 0.0 0.0 1.0"/>
+</material>
+<material name="blue">
+  <color rgba="0.0 0.0 0.8 1.0"/>
+</material>
+<material name="green">
+  <color rgba="0.0 0.8 0.0 1.0"/>
+</material>
+<material name="grey">
+  <color rgba="0.2 0.2 0.2 1.0"/>
+</material>
+<material name="orange">
+  <color rgba="${255/255} ${108/255} ${10/255} 1.0"/>
+</material>
+<material name="brown">
+  <color rgba="${222/255} ${207/255} ${195/255} 1.0"/>
+</material>
+<material name="red">
+  <color rgba="0.8 0.0 0.0 1.0"/>
+</material>
+<material name="white">
+  <color rgba="1.0 1.0 1.0 1.0"/>
+</material>
 </robot>

File: src/ogmen_description/urdf/ogmen.xacro (robot description, xacro)
@@ -15,5 +15,5 @@
       <mesh filename="file://$(find ogmen_description)/meshes/base_link.stl" scale="0.001 0.001 0.001"/>
     </geometry>
-    <material name="silver"/>
+    <material name="blue"/>
   </visual>
   <collision>
@@ -35,5 +35,5 @@
       <mesh filename="file://$(find ogmen_description)/meshes/right_wheel_1.stl" scale="0.001 0.001 0.001"/>
     </geometry>
-    <material name="silver"/>
+    <material name="black"/>
   </visual>
   <collision>
@@ -55,5 +55,5 @@
       <mesh filename="file://$(find ogmen_description)/meshes/left_wheel_1.stl" scale="0.001 0.001 0.001"/>
     </geometry>
-    <material name="silver"/>
+    <material name="black"/>
   </visual>
   <collision>
@@ -75,5 +75,5 @@
       <mesh filename="file://$(find ogmen_description)/meshes/lidar_1.stl" scale="0.001 0.001 0.001"/>
     </geometry>
-    <material name="silver"/>
+    <material name="orange"/>
   </visual>
   <collision>
@@ -104,11 +104,11 @@
   </collision>
 </link>
-<joint name="Revolute 1" type="continuous">
+<joint name="right_wheel_joint" type="continuous">
   <origin xyz="-0.035 -0.105 0.065" rpy="0 0 0"/>
   <parent link="base_link"/>
   <child link="right_wheel_1"/>
-  <axis xyz="0.0 -1.0 0.0"/>
+  <axis xyz="0.0 1.0 0.0"/>
 </joint>
-<joint name="Revolute 2" type="continuous">
+<joint name="left_wheel_joint" type="continuous">
   <origin xyz="-0.035 0.105 0.065" rpy="0 0 0"/>
   <parent link="base_link"/>
@@ -116,10 +116,10 @@
   <axis xyz="0.0 1.0 0.0"/>
 </joint>
-<joint name="Rigid 3" type="fixed">
+<joint name="Lidar_joint" type="fixed">
   <origin xyz="0.0 0.0 0.135" rpy="0 0 0"/>
   <parent link="base_link"/>
   <child link="lidar_1"/>
 </joint>
-<joint name="Rigid 4" type="fixed">
+<joint name="Camera_joint" type="fixed">
   <origin xyz="0.1 0.0 0.08" rpy="0 0 0"/>
   <parent link="base_link"/>
